File: display/board/hp3478-display/hp3478-display.kicad_pcb (KiCad board)
At the start: 2 copper layers, 130.2 x 29.8 mm, 245 parts, among them J1 Header, J2 Header, U1 FT60F1x2, U2 SM16206, U3 74HC595, U4 74HC595

Commit message: Choose LEDs and set drive current.
Parts:
- added R1: 5k6 1%, Resistor_SMD:R_0603_1608Metric, F.Cu at (90.7, 71.9)
- U2: value SM16206 -> SM16206S
Connections:
- U2 pad 23: unconnected-(U2-Pad23) -> Net-(U2-Pad23)
Routing:
- net GND: track 193.4 -> 198.8 mm
- net Net-(U2-Pad23): track 0.00 -> 2.50 mm

Commit message: Swap LCD_P1 and LCD_PWO on MCU so P1 can have edge-triggered interrupts.
Connections:
- U1 pad 10: /LCD_P1 -> /LCD_PWO
- U1 pad 11: /LCD_PWO -> /LCD_P1
Routing:
- net /LCD_P1: track 68.0 -> 65.8 mm
- net /LCD_PWO: track 62.9 -> 62.0 mm
Changed lines of the file:
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@@
       (net 35 "/DSD") (pinfunction "PC0") (pintype "bidirectional"))
     (pad "10" smd roundrect (at 2.475 1.27 270) (size 1.95 0.6) (layers "F.Cu" "F.Paste" "F.Mask") (roundrect_rratio 0.25)
-      (net 51 "/LCD_P1") (pinfunction "PA3") (pintype "bidirectional"))
+      (net 50 "/LCD_PWO") (pinfunction "PA3") (pintype "bidirectional"))
     (pad "11" smd roundrect (at 2.475 0 270) (size 1.95 0.6) (layers "F.Cu" "F.Paste" "F.Mask") (roundrect_rratio 0.25)
-      (net 50 "/LCD_PWO") (pinfunction "PA2/T0CKI/INT") (pintype "bidirectional"))
+      (net 51 "/LCD_P1") (pinfunction "PA2/T0CKI/INT") (pintype "bidirectional"))
     (pad "12" smd roundrect (at 2.475 -1.27 270) (size 1.95 0.6) (layers "F.Cu" "F.Paste" "F.Mask") (roundrect_rratio 0.25)
       (net 20 "/PGD") (pinfunction "ISPDAT/PA1") (pintype "bidirectional"))
@@
   (segment (start 162.9893 64.0563) (end 162.9893 52.7911) (width 0.127) (layer "B.Cu") (net 42))
   (segment (start 122.656951 68.999053) (end 123.6525 68.003504) (width 0.127) (layer "B.Cu") (net 42))
-  (segment (start 194.31 75.692) (end 194.31 68.515) (width 0.127) (layer "F.Cu") (net 50))
-  (segment (start 191.008 78.994) (end 194.31 75.692) (width 0.127) (layer "F.Cu") (net 50))
-  (segment (start 157.734 78.994) (end 191.008 78.994) (width 0.127) (layer "F.Cu") (net 50))
-  (segment (start 151.13 72.39) (end 157.734 78.994) (width 0.127) (layer "F.Cu") (net 50))
-  (segment (start 151.13 65.786) (end 151.13 72.39) (width 0.127) (layer "F.Cu") (net 50))
-  (segment (start 149.86 64.516) (end 151.13 65.786) (width 0.127) (layer "F.Cu") (net 50))
-  (segment (start 148.844 60.96) (end 150.368 60.96) (width 0.127) (layer "F.Cu") (net 51))
-  (segment (start 190.754 78.486) (end 193.04 76.2) (width 0.127) (layer "F.Cu") (net 51))
-  (segment (start 150.368 60.96) (end 151.638 62.23) (width 0.127) (layer "F.Cu") (net 51))
-  (segment (start 151.638 62.23) (end 151.638 72.136) (width 0.127) (layer "F.Cu") (net 51))
-  (segment (start 193.04 76.2) (end 193.04 68.515) (width 0.127) (layer "F.Cu") (net 51))
-  (segment (start 147.32 62.484) (end 148.844 60.96) (width 0.127) (layer "F.Cu") (net 51))
-  (segment (start 151.638 72.136) (end 157.988 78.486) (width 0.127) (layer "F.Cu") (net 51))
-  (segment (start 157.988 78.486) (end 190.754 78.486) (width 0.127) (layer "F.Cu") (net 51))
+  (segment (start 151.638 72.136) (end 151.638 66.294) (width 0.127) (layer "F.Cu") (net 50))
+  (segment (start 190.754 78.486) (end 157.988 78.486) (width 0.127) (layer "F.Cu") (net 50))
+  (segment (start 149.86 64.516) (end 149.86 63.515) (width 0.127) (layer "F.Cu") (net 50))
+  (segment (start 157.988 78.486) (end 151.638 72.136) (width 0.127) (layer "F.Cu") (net 50))
+  (segment (start 193.04 76.2) (end 190.754 78.486) (width 0.127) (layer "F.Cu") (net 50))
+  (segment (start 193.04 68.515) (end 193.04 76.2) (width 0.127) (layer "F.Cu") (net 50))
+  (segment (start 151.638 66.294) (end 149.86 64.516) (width 0.127) (layer "F.Cu") (net 50))
+  (segment (start 150.368 66.04) (end 148.844 66.04) (width 0.127) (layer "F.Cu") (net 51))
+  (segment (start 194.31 68.515) (end 194.31 75.692) (width 0.127) (layer "F.Cu") (net 51))
+  (segment (start 194.31 75.692) (end 191.008 78.994) (width 0.127) (layer "F.Cu") (net 51))
+  (segment (start 148.844 66.04) (end 147.32 64.516) (width 0.127) (layer "F.Cu") (net 51))
+  (segment (start 151.13 66.802) (end 150.368 66.04) (width 0.127) (layer "F.Cu") (net 51))
+  (segment (start 147.32 64.516) (end 147.32 63.515) (width 0.127) (layer "F.Cu") (net 51))
+  (segment (start 191.008 78.994) (end 157.734 78.994) (width 0.127) (layer "F.Cu") (net 51))
+  (segment (start 157.734 78.994) (end 151.13 72.39) (width 0.127) (layer "F.Cu") (net 51))
+  (segment (start 151.13 72.39) (end 151.13 66.802) (width 0.127) (layer "F.Cu") (net 51))
   (segment (start 187.96 70.104) (end 187.96 63.5) (width 0.127) (layer "F.Cu") (net 53))
   (segment (start 152.146 71.882) (end 158.242 77.978) (width 0.127) (layer "F.Cu") (net 53))
